Commit message: Add files via upload

File: basic_amr_description/urdf/basic_amr.xacro (robot description, xacro)
@@ -14,10 +14,11 @@
   </material>
   <!-- Begin - Robot description -->
-  <link name="base_link" />
-  <joint name="base__base_link" type="fixed">
-    <parent link="base_link"/>
-    <child link="base"/>
+  <link name="base_footprint" />
+  <joint name="base_link__base_footprint" type="fixed">
+    <parent link="base_footprint"/>
+    <child link="base_link"/>
+    <origin xyz="0.0 0.0 0.003" rpy="0 0 0"/>
   </joint>
-  <link name="base">
+  <link name="base_link">
     <origin rpy="0 0 0" xyz="0.00 0 0.00"/>
     <visual>
@@ -41,5 +42,5 @@
     <visual>
       <geometry>
-        <cylinder length="0.006" radius="0.0035"/>
+        <sphere radius="0.0035"/>
       </geometry>
       <material name="black"/>
@@ -47,17 +48,17 @@
     <collision>
       <geometry>
-        <cylinder length="0.006" radius="0.0035"/>
+        <sphere radius="0.0035"/>
       </geometry>
     </collision>
     <inertial>
-      <mass value="0.05" />
+      <origin xyz="0 0 0" />
+      <mass value="0.01" />
       <inertia ixx="0.001" ixy="0.0" ixz="0.0" iyy="0.001" iyz="0.0" izz="0.001" />
     </inertial>
   </link>
-  <joint name="base__fcastor_wheel" type="continuous">
-    <parent link="base"/>
+  <joint name="base_link__fcastor_wheel" type="fixed">
+    <parent link="base_link"/>
     <child link="fcastor_wheel"/>
     <origin xyz="0.028 0 -0.005" rpy="1.5708 0 0"/>
-    <axis xyz="0 0 1"/>
   </joint>
   <link name="bcastor_wheel">
@@ -65,5 +66,5 @@
     <visual>
       <geometry>
-        <cylinder length="0.006" radius="0.0035"/>
+        <sphere radius="0.0035"/>
       </geometry>
       <material name="black"/>
@@ -71,17 +72,17 @@
     <collision>
       <geometry>
-        <cylinder length="0.006" radius="0.0035"/>
+        <sphere radius="0.0035"/>
       </geometry>
     </collision>
     <inertial>
-      <mass value="0.05" />
+      <origin xyz="0 0 0" />
+      <mass value="0.01" />
       <inertia ixx="0.001" ixy="0.0" ixz="0.0" iyy="0.001" iyz="0.0" izz="0.001" />
     </inertial>
   </link>
-  <joint name="base__bcastor_wheel" type="continuous">
-    <parent link="base"/>
+  <joint name="base_link__bcastor_wheel" type="fixed">
+    <parent link="base_link"/>
     <child link="bcastor_wheel"/>
     <origin xyz="-0.028 0 -0.005" rpy="1.5708 0 0"/>
-    <axis xyz="0 0 1"/>
   </joint>
   <link name="left_wheel">
@@ -104,5 +105,5 @@
   </link>
   <joint name="wheel_left_joint" type="continuous">
-    <parent link="base"/>
+    <parent link="base_link"/>
     <child link="left_wheel"/>
     <origin xyz="0 0.032 0.007" rpy="1.5708 0 0"/>
@@ -128,5 +129,5 @@
   </link>
   <joint name="wheel_right_joint" type="continuous">
-    <parent link="base"/>
+    <parent link="base_link"/>
     <child link="right_wheel"/>
     <origin xyz="0 -0.032 0.007" rpy="1.5708 0 0"/>
@@ -145,11 +146,11 @@
     </visual>
   </link>
-  <joint name="base__front_camera_joint" type="fixed">
-    <parent link="base"/>
+  <joint name="base_link__front_camera" type="fixed">
+    <parent link="base_link"/>
     <child link="front_camera_link"/>
     <origin xyz="0.040 0 0" rpy="0 0 0"/>
   </joint>
   <!-- 2D Lidar representation -->
-  <link name="rplidar_link">
+  <link name="base_scan">
     <visual>
       <origin rpy="0.0 0 0" xyz="0 0 0"/>
@@ -160,7 +161,7 @@
     </visual>
   </link>
-  <joint name="base__rplidar_link_joint" type="fixed">
-    <parent link="base"/>
-    <child link="rplidar_link"/>
+  <joint name="base_link__base_scan" type="fixed">
+    <parent link="base_link"/>
+    <child link="base_scan"/>
     <origin xyz="0 0 0.03" rpy="0 0 0"/>
   </joint>

File: basic_amr_description/urdf/basic_amr_gazebo.xacro (robot description, xacro)
@@ -2,10 +2,10 @@
 <robot name="basic_amr" xmlns:xacro="http://ros.org/wiki/xacro">
   <!-- Begin - Gazebo definition -->
-  <gazebo reference="base">
+  <gazebo reference="base_link">
     <material>Gazebo/White</material>
   </gazebo>
   <gazebo reference="right_wheel">
-    <mu1>0.5</mu1>
-    <mu2>0.5</mu2>
+    <mu1>0.1</mu1>
+    <mu2>0.1</mu2>
     <kp>500000.0</kp>
     <kd>10.0</kd>
@@ -16,6 +16,6 @@
   </gazebo>
   <gazebo reference="left_wheel">
-    <mu1>0.5</mu1>
-    <mu2>0.5</mu2>
+    <mu1>0.1</mu1>
+    <mu2>0.1</mu2>
     <kp>500000.0</kp>
     <kd>10.0</kd>
@@ -26,21 +26,19 @@
   </gazebo>
   <gazebo reference="fcastor_wheel">
-    <mu1>0.5</mu1>
-    <mu2>0.5</mu2>
-    <kp>500000.0</kp>
-    <kd>10.0</kd>
+    <mu1>0.1</mu1>
+    <mu2>0.1</mu2>
+    <kp>1000000.0</kp>
+    <kd>100.0</kd>
     <minDepth>0.001</minDepth>
-    <maxVel>0.1</maxVel>
-    <fdir1>1 0 0</fdir1>
+    <maxVel>1.0</maxVel>
     <material>Gazebo/FlatBlack</material>
   </gazebo>
   <gazebo reference="bcastor_wheel">
-    <mu1>0.5</mu1>
-    <mu2>0.5</mu2>
-    <kp>500000.0</kp>
-    <kd>10.0</kd>
+    <mu1>0.1</mu1>
+    <mu2>0.1</mu2>
+    <kp>1000000.0</kp>
+    <kd>100.0</kd>
     <minDepth>0.001</minDepth>
-    <maxVel>0.1</maxVel>
-    <fdir1>1 0 0</fdir1>
+    <maxVel>1.0</maxVel>
     <material>Gazebo/FlatBlack</material>
   </gazebo>
@@ -54,14 +52,16 @@
       <wheelDiameter>0.032</wheelDiameter>
       <wheelAcceleration>0.1</wheelAcceleration>
-      <wheelTorque>20</wheelTorque>
+      <wheelTorque>10</wheelTorque>
       <commandTopic>cmd_vel</commandTopic>
       <odometryTopic>odom</odometryTopic>
       <odometryFrame>odom</odometryFrame>
+      <odometrySource>world</odometrySource>
       <robotBaseFrame>base_footprint</robotBaseFrame>
-      <publishWheelTF>true</publishWheelTF>
-      <publishOdom>true</publishOdom>
-      <robotBaseFrame>base</robotBaseFrame>
+      <publishTF>true</publishTF>
+      <publishOdomTF>true</publishOdomTF>
+      <publishWheelTF>false</publishWheelTF>
       <publishWheelJointState>true</publishWheelJointState>
       <legacyMode>false</legacyMode>
+      <rosDebugLevel>na</rosDebugLevel>
     </plugin>
   </gazebo>
@@ -109,9 +109,9 @@
     </sensor>
   </gazebo>
-  <gazebo reference="laser_link">
+  <gazebo reference="base_scan">
     <material>Gazebo/Yellow</material>
   </gazebo>
   <!-- 2D Lidar plugin for gazebo -->
-  <gazebo reference="rplidar_link">
+  <gazebo reference="base_scan">
     <sensor type="ray" name="rplidar_sensor">
       <pose>0 0 0 0 0 0</pose>
@@ -139,6 +139,6 @@
       </ray>
       <plugin name="gazebo_ros_head_hokuyo_controller" filename="libgazebo_ros_laser.so">
-        <topicName>/laser_scan</topicName>
-        <frameName>rplidar_link</frameName>
+        <topicName>/scan</topicName>
+        <frameName>base_scan</frameName>
       </plugin>
     </sensor>

Commit message: Add files via upload

File: basic_amr_description/urdf/basic_amr.xacro (robot description, xacro)
@@ -34,6 +34,6 @@
     </collision>
     <inertial>
-      <mass value="0.5" />
-      <inertia ixx="1.0" ixy="0.0" ixz="0.0" iyy="1.0" iyz="0.0" izz="1.0" />
+      <mass value="0.2" />
+      <inertia ixx="0.1" ixy="0.0" ixz="0.0" iyy="0.1" iyz="0.0" izz="0.1" />
     </inertial>
   </link>
@@ -53,6 +53,6 @@
     <inertial>
       <origin xyz="0 0 0" />
-      <mass value="0.01" />
-      <inertia ixx="0.001" ixy="0.0" ixz="0.0" iyy="0.001" iyz="0.0" izz="0.001" />
+      <mass value="0.002" />
+      <inertia ixx="0.0001" ixy="0.0" ixz="0.0" iyy="0.0001" iyz="0.0" izz="0.0001" />
     </inertial>
   </link>
@@ -77,6 +77,6 @@
     <inertial>
       <origin xyz="0 0 0" />
-      <mass value="0.01" />
-      <inertia ixx="0.001" ixy="0.0" ixz="0.0" iyy="0.001" iyz="0.0" izz="0.001" />
+      <mass value="0.002" />
+      <inertia ixx="0.0001" ixy="0.0" ixz="0.0" iyy="0.0001" iyz="0.0" izz="0.0001" />
     </inertial>
   </link>
@@ -100,5 +100,5 @@
     </collision>
     <inertial>
-      <mass value="0.05" />
+      <mass value="0.02" />
       <inertia ixx="0.001" ixy="0.0" ixz="0.0" iyy="0.001" iyz="0.0" izz="0.001" />
     </inertial>
@@ -124,5 +124,5 @@
     </collision>
     <inertial>
-      <mass value="0.05" />
+      <mass value="0.02" />
       <inertia ixx="0.001" ixy="0.0" ixz="0.0" iyy="0.001" iyz="0.0" izz="0.001" />
     </inertial>
